Commit message: 这是第一个launch文件

File: src/lykbot_dstion/urdf/fishbot.urdf (robot description, URDF)
Before this commit: robot fishrobot, 1 links, 0 joints
Links:
- added link imu_link; visual box size=0.02 0.02 0.02
Joints:
- added joint imu_name: type fixed, parent base_link, child imu_link, origin xyz=0.0 0.0 0.05 rpy=0.0 0.0 0.0

Commit message: 这里包含车身配件的】xacro文件

File: src/lykbot_dstion/urdf/fishbot.urdf (robot description, URDF)
Before this commit: robot fishrobot, 2 links, 1 joints
Joints:
- removed joint imu_name
- added joint imu_joint: type fixed, parent base_link, child imu_link, origin xyz=0.0 0.0 0.03 rpy=0.0 0.0 0.0
