Commit message: 这是包含了碰撞部分的

File: src/lykbot_dstion/urdf/lykbot/base.urdf.xacro (robot description, xacro)
@@ -2,4 +2,5 @@
 <robot xmlns:xacro="http://www.ros.org/wiki/xacro">
     <xacro:macro name = "base_xacro" params="length radius">
+        <link name="base_footprint" />
             <!-- 机器人身体的部分-->
         <link name="base_link">
@@ -18,4 +19,9 @@
             </visual>
         </link>
+        <joint name="joint_name" type="fixed">
+            <origin xyz="0.0 0.0 ${length/2.0+0.032-0.001}" rpy="0.0 0.0 0.0"/>
+            <parent link="base_footprint"/>
+            <child link="base_link"/>
+        </joint>
     </xacro:macro>
 </robot>

File: src/lykbot_dstion/urdf/lykbot/lykbot.urdf.xacro (robot description, xacro)
@@ -6,4 +6,10 @@
 <xacro:include filename="$(find lykbot_dstion)/urdf/lykbot/sensor/camera.urdf.xacro"/>
 <xacro:include filename="$(find lykbot_dstion)/urdf/lykbot/sensor/laser.urdf.xacro"/>
+<xacro:include filename="$(find lykbot_dstion)/urdf/lykbot/actuator/wheel.urdf.xacro"/>
+<xacro:include filename="$(find lykbot_dstion)/urdf/lykbot/actuator/caster.urdf.xacro"/>
+<xacro:wheel_xacro wheel_name="left_wheel" xyz="0 0.10 -0.06"/>
+<xacro:wheel_xacro wheel_name="right_wheel" xyz="0 -0.10 -0.06"/>
+<xacro:caster_xacro caster_name="left_caster" xyz="0.08 0.0 -0.076"/>
+<xacro:caster_xacro caster_name="right_caster" xyz="-0.08 0.0 -0.076"/>
 <xacro:base_xacro length="0.12" radius="0.10"/>
 <xacro:imu_xacro xyz="0.0 0.0 0.02"/>
