Commit message: 添加了质量的属性

File: src/lykbot_dstion/urdf/lykbot/actuator/caster.urdf.xacro (robot description, xacro)
@@ -1,4 +1,5 @@
 <?xml version="1.0"?>
 <robot xmlns:xacro="http://www.ros.org/wiki/xacro">
+   <xacro:include filename="$(find lykbot_dstion)/urdf/lykbot/common_inertia.xacro"/>
   <xacro:macro name = "caster_xacro" params="caster_name xyz">
    <!-- 这是机器人的imu部件 -->
@@ -17,4 +18,17 @@
             </material>
         </visual>
+        <collision>
+                        <!-- 沿着自己几何中心的偏移量 -->
+            <origin xyz="0.0 0.0 0.0" rpy="0.0 0.0 0.0"/>
+            <!-- 几何形状 -->
+            <geometry>
+            <!-- 这是一个正方体 -->
+               <sphere radius="0.016"/>
+            </geometry>
+            <!-- 这是材质和颜色的描述 -->
+            <material name="yellow">
+                <color rgba="1.0 1.0 1.0 0.5"/>
+            </material>
+        </collision>
     </link>
      <joint name="${caster_name}_joint" type="fixed">
@@ -23,4 +37,6 @@
         <child link="${caster_name}_link"/>
     </joint>
+     <!-- 描述质量和惯性的 -->
+    <xacro:sphere_inertia m="0.05" r="0.016" />
   </xacro:macro>
 </robot>

File: src/lykbot_dstion/urdf/lykbot/actuator/wheel.urdf.xacro (robot description, xacro)
@@ -1,4 +1,5 @@
 <?xml version="1.0"?>
 <robot xmlns:xacro="http://www.ros.org/wiki/xacro">
+  <xacro:include filename="$(find lykbot_dstion)/urdf/lykbot/common_inertia.xacro"/>
   <xacro:macro name = "wheel_xacro" params="wheel_name xyz">
    <!-- 这是机器人的imu部件 -->
@@ -17,4 +18,18 @@
             </material>
         </visual>
+        <collision>
+                      <!-- 沿着自己几何中心的偏移量 -->
+            <origin xyz="0.0 0.0 0.0" rpy="1.59079 0.0 0.0"/>
+            <!-- 几何形状 -->
+            <geometry>
+            <!-- 这是一个正方体 -->
+               <cylinder radius="0.032" length="0.03"/>
+            </geometry>
+            <!-- 这是材质和颜色的描述 -->
+            <material name="yellow">
+                <color rgba="1.0 1.0 1.0 0.5"/>
+            </material>
+        </collision>
+        <xacro:cylinder_inertia m="0.05" r="0.032" h="0.03"/>
     </link>
      <joint name="${wheel_name}_joint" type="continuous">

File: src/lykbot_dstion/urdf/lykbot/base.urdf.xacro (robot description, xacro)
@@ -1,4 +1,5 @@
 <?xml version="1.0"?>
 <robot xmlns:xacro="http://www.ros.org/wiki/xacro">
+    <xacro:include filename="$(find lykbot_dstion)/urdf/lykbot/common_inertia.xacro"/>
     <xacro:macro name = "base_xacro" params="length radius">
         <link name="base_footprint" />
@@ -18,4 +19,19 @@
                 </material>
             </visual>
+            <collision>
+                 <!-- 沿着自己几何中心的偏移量 -->
+                <origin xyz="0.0 0.0 0.0" rpy="0.0 0.0 0.0"/>
+                <!-- 几何形状 -->
+                <geometry>
+                <!-- 这是一个圆柱体，半径为10cm，高度为12cm -->
+                    <cylinder radius="${radius}" length="${length}"/>
+                </geometry>
+                <!-- 这是材质和颜色的描述 -->
+                <material name="white">
+                    <color rgba="1.0 1.0 1.0 0.5"/>
+                </material>
+            </collision>
+            <!-- 描述质量和惯性的 -->
+            <xacro:cylinder_inertia m="1.0" r="${radius}" h="${length}"/>
         </link>
         <joint name="joint_name" type="fixed">

File: src/lykbot_dstion/urdf/lykbot/sensor/camera.urdf.xacro (robot description, xacro)
@@ -1,4 +1,5 @@
 <?xml version="1.0"?>
 <robot xmlns:xacro="http://www.ros.org/wiki/xacro">
+<xacro:include filename="$(find lykbot_dstion)/urdf/lykbot/common_inertia.xacro"/>
   <xacro:macro name = "camera_xacro" params="xyz">
    <!-- 这是机器人的摄像头的部件 -->
@@ -17,4 +18,19 @@
             </material>
         </visual>
+        <collision>
+            <!-- 沿着自己几何中心的偏移量 -->
+            <origin xyz="0.0 0.0 0.0" rpy="0.0 0.0 0.0"/>
+            <!-- 几何形状 -->
+            <geometry>
+            <!-- 这是一个正方体 -->
+                <box size="0.02 0.10 0.02"/>
+            </geometry>
+            <!-- 这是材质和颜色的描述 -->
+            <material name="black">
+                <color rgba="0.0 0.0 0.0 0.5"/>
+            </material>
+        </collision>
+         <!-- 描述质量和惯性的 -->
+            <xacro:box_inertia m="0.1" w="0.02" h="0.10" d="0.12"/>
     </link>
      <joint name="camera_joint" type="fixed">

File: src/lykbot_dstion/urdf/lykbot/sensor/imu.urdf.xacro (robot description, xacro)
@@ -1,4 +1,5 @@
 <?xml version="1.0"?>
 <robot xmlns:xacro="http://www.ros.org/wiki/xacro">
+   <xacro:include filename="$(find lykbot_dstion)/urdf/lykbot/common_inertia.xacro"/>
   <xacro:macro name = "imu_xacro" params="xyz">
    <!-- 这是机器人的imu部件 -->
@@ -17,4 +18,19 @@
             </material>
         </visual>
+        <collision>
+            <!-- 沿着自己几何中心的偏移量 -->
+            <origin xyz="0.0 0.0 0.0" rpy="0.0 0.0 0.0"/>
+            <!-- 几何形状 -->
+            <geometry>
+            <!-- 这是一个正方体 -->
+                <box size="0.02 0.02 0.02"/>
+            </geometry>
+            <!-- 这是材质和颜色的描述 -->
+            <material name="black">
+                <color rgba="0.0 0.0 0.0 0.5"/>
+            </material>
+        </collision>
+         <!-- 描述质量和惯性的 -->
+            <xacro:box_inertia m="0.05" w="0.02" h="0.02" d="0.02"/>
     </link>
      <joint name="imu_joint" type="fixed">

File: src/lykbot_dstion/urdf/lykbot/sensor/laser.urdf.xacro (robot description, xacro)
@@ -1,4 +1,5 @@
 <?xml version="1.0"?>
 <robot xmlns:xacro="http://www.ros.org/wiki/xacro">
+<xacro:include filename="$(find lykbot_dstion)/urdf/lykbot/common_inertia.xacro"/>
   <xacro:macro name = "laser_xacro" params="xyz">
   <!-- 这是雷达的支撑杆 -->
@@ -17,4 +18,19 @@
             </material>
         </visual>
+        <collision>
+             <!-- 沿着自己几何中心的偏移量 -->
+            <origin xyz="0.0 0.0 0.0" rpy="0.0 0.0 0.0"/>
+            <!-- 几何形状 -->
+            <geometry>
+            <!-- 这是一个圆柱 -->
+                <cylinder radius="0.01" length="0.10"/>
+            </geometry>
+            <!-- 这是材质和颜色的描述 -->
+            <material name="black">
+                <color rgba="0.0 0.0 0.0 1.0"/>
+            </material>
+        </collision>
+                 <!-- 描述质量和惯性的 -->
+            <xacro:cylinder_inertia m="0.05" r="0.01" h="0.10"/>
     </link>
     <!-- 这是机器人的雷达的部件 -->
@@ -33,4 +49,19 @@
             </material>
         </visual>
+        <collision>
+                       <!-- 沿着自己几何中心的偏移量 -->
+            <origin xyz="0.0 0.0 0.0" rpy="0.0 0.0 0.0"/>
+            <!-- 几何形状 -->
+            <geometry>
+            <!-- 这是一个圆柱-->
+                <cylinder radius="0.02" length="0.02"/>
+            </geometry>
+            <!-- 这是材质和颜色的描述 -->
+            <material name="black">
+                <color rgba="0.0 0.0 0.0 1.0"/>
+            </material>
+        </collision>
+                 <!-- 描述质量和惯性的 -->
+            <xacro:cylinder_inertia m="0.05" r="0.02" h="0.02"/>
     </link>
     <joint name="laser_cylinder_joint" type="fixed">
